File: ide_adapter.kicad_pcb (KiCad board)
At the start: 2 copper layers, 42 x 46 mm, 15 parts, among them J1 PATA-44_Host, J2 Conn_01x06_Male, J3 PATA-44_Drive, J4 PATA-44_Drive, U1 LM1117-3.3, U2 LT1129-3.3_SOT223, U3 XC9572XL-VQ64

Commit message: Version 1 as ordered
Routing:
- net GND: track 123.5 -> 157.1 mm, vias 12 -> 15
- net /TCK: track 16.0 -> 23.7 mm, vias 1 -> 3
- net +3V3: track 92.9 -> 91.0 mm, vias 5 -> 4
- net /~RESET: track 76.4 -> 77.7 mm
- net /TDO: track 21.6 -> 22.4 mm
- net /TMS: track 18.9 -> 19.6 mm

Commit message: Adding silkscreen for release.
Other:
- board text added: "3V3 REG CENTRE=3V3"
- board text added: "3V3 REG CENTRE=GND"
- board text added: "ALL CAPS 100n"
- board text added: "Copyright 2023 D Henderson GPLv2 github.com/dh219 @thetechnoshed"
- board text added: "FIT ONLY ONE REGULATOR"
- board text added: "MASTER (CS)"
- board text added: "SLAVE (CS)"
- board text added: "~DAVID'S AUTO-SWAPPING FALCON IDE ADAPTER"
- board text removed: "MASTER"
- board text removed: "SLAVE"
